Commit message: add rviz visualization and rviz config

File: uthai_description/urdf/uthai.xacro (robot description, xacro)
@@ -6,4 +6,5 @@
     <xacro:include filename="$(find uthai_description)/urdf/materials.xacro" />
     <xacro:include filename="$(find uthai_description)/urdf/uthai_leg.xacro" />
+    <xacro:include filename="$(find uthai_description)/urdf/uthai.gazebo" />
     <!-- Used for fixing robot -->
     <link name="world"></link>

File: uthai_description/urdf/uthai_leg.xacro (robot description, xacro)
@@ -183,4 +183,12 @@
             </inertial>
         </link>
+        <!-- left ft fixed joint -->
+        <joint name="l_ft_fixed" type="fixed">
+            <origin xyz="0.05 0.0 0.0" rpy="0 ${-pi/2} 0"/>
+            <parent link="l_ankle_roll_link"/>
+            <child link="l_foot_ft_link"/>
+        </joint>
+        <!-- left foot ft link -->
+        <link name="l_foot_ft_link"></link>
     </xacro:macro>
     <xacro:macro name="uthai_right_leg" params="parent">
@@ -353,4 +361,12 @@
             </inertial>
         </link>
+        <!-- right ft fixed joint -->
+        <joint name="r_ft_fixed" type="fixed">
+            <origin xyz="0.05 0.0 0.0" rpy="0 ${-pi/2} 0"/>
+            <parent link="r_ankle_roll_link"/>
+            <child link="r_foot_ft_link"/>
+        </joint>
+        <!-- right foot ft link -->
+        <link name="r_foot_ft_link"></link>
     </xacro:macro>
 </robot>

Commit message: update xacro files

File: uthai_description/urdf/uthai.xacro (robot description, xacro)
@@ -8,5 +8,5 @@
     <xacro:include filename="$(find uthai_description)/urdf/uthai.gazebo" />
     <!-- Used for fixing robot -->
-    <link name="world"></link>
+    <!--<link name="world"></link>
     <joint name="world_fixed" type="fixed">
         <origin xyz="0 0 0.756" rpy="0 0 0"/>
@@ -19,5 +19,5 @@
         <parent link="base"/>
         <child link="pelvis_link"/>
-    </joint>
+    </joint>-->
     <!-- pelvis_link -->
     <link name="pelvis_link">

File: uthai_description/urdf/uthai_leg.xacro (robot description, xacro)
@@ -21,5 +21,5 @@
             <parent link="${parent}"/>
             <child link="l_hip_yaw_link"/>
-            <limit effort="10" lower="${-pi*0.9}" upper="${pi*0.9}" velocity="5.6548668"/>
+            <limit effort="20" lower="${-pi*0.9}" upper="${pi*0.9}" velocity="10"/>
             <dynamics damping="0.1" friction="0.0"/>
         </joint>
@@ -49,5 +49,5 @@
             <parent link="l_hip_yaw_link"/>
             <child link="l_hip_roll_link"/>
-            <limit effort="10" lower="${-pi*0.9}" upper="${pi*0.9}" velocity="5.6548668"/>
+            <limit effort="20" lower="${-pi*0.9}" upper="${pi*0.9}" velocity="10"/>
             <dynamics damping="0.1" friction="0.0"/>
         </joint>
@@ -77,5 +77,5 @@
             <parent link="l_hip_roll_link"/>
             <child link="l_hip_pitch_link"/>
-            <limit effort="10" lower="${-pi*0.9}" upper="${pi*0.9}" velocity="5.6548668"/>
+            <limit effort="20" lower="${-pi*0.9}" upper="${pi*0.9}" velocity="10"/>
             <dynamics damping="0.1" friction="0.0"/>
         </joint>
@@ -105,5 +105,5 @@
             <parent link="l_hip_pitch_link"/>
             <child link="l_knee_pitch_link"/>
-            <limit effort="10" lower="${-pi*0.9}" upper="${pi*0.9}" velocity="5.6548668"/>
+            <limit effort="20" lower="${-pi*0.9}" upper="${pi*0.9}" velocity="10"/>
             <dynamics damping="0.1" friction="0.0"/>
         </joint>
@@ -133,5 +133,5 @@
             <parent link="l_knee_pitch_link"/>
             <child link="l_ankle_pitch_link"/>
-            <limit effort="10" lower="${-pi*0.9}" upper="${pi*0.9}" velocity="5.6548668"/>
+            <limit effort="20" lower="${-pi*0.9}" upper="${pi*0.9}" velocity="10"/>
             <dynamics damping="0.1" friction="0.0"/>
         </joint>
@@ -161,5 +161,5 @@
             <parent link="l_ankle_pitch_link"/>
             <child link="l_ankle_roll_link"/>
-            <limit effort="10" lower="${-pi*0.9}" upper="${pi*0.9}" velocity="5.6548668"/>
+            <limit effort="20" lower="${-pi*0.9}" upper="${pi*0.9}" velocity="10"/>
             <dynamics damping="0.1" friction="0.0"/>
         </joint>
@@ -178,7 +178,7 @@
             </visual>
             <inertial>
-                <origin xyz="0.03576926 -0.08779574 -0.00045842"/>
+                           <origin xyz="0.03625957 -0.00019537 0.00037602"/>
                 <mass value="0.10500000"/>
-                <inertia ixx="0.00123572" ixy="0.00000500" ixz="0.00000812" iyy="0.00031773" iyz="0.00000828" izz="0.00094763" />
+                <inertia ixx="0.00034590" ixy="-0.00000013" ixz="0.00000857" iyy="0.00032704" iyz="0.00000120" izz="0.00004812" />
             </inertial>
         </link>
@@ -199,5 +199,5 @@
             <parent link="${parent}"/>
             <child link="r_hip_yaw_link"/>
-            <limit effort="10" lower="${-pi*0.9}" upper="${pi*0.9}" velocity="5.6548668"/>
+            <limit effort="20" lower="${-pi*0.9}" upper="${pi*0.9}" velocity="10"/>
             <dynamics damping="0.1" friction="0.0"/>
         </joint>
@@ -227,5 +227,5 @@
             <parent link="r_hip_yaw_link"/>
             <child link="r_hip_roll_link"/>
-            <limit effort="10" lower="${-pi*0.9}" upper="${pi*0.9}" velocity="5.6548668"/>
+            <limit effort="20" lower="${-pi*0.9}" upper="${pi*0.9}" velocity="10"/>
             <dynamics damping="0.1" friction="0.0"/>
         </joint>
@@ -255,5 +255,5 @@
             <parent link="r_hip_roll_link"/>
             <child link="r_hip_pitch_link"/>
-            <limit effort="10" lower="${-pi*0.9}" upper="${pi*0.9}" velocity="5.6548668"/>
+            <limit effort="20" lower="${-pi*0.9}" upper="${pi*0.9}" velocity="10"/>
             <dynamics damping="0.1" friction="0.0"/>
         </joint>
@@ -283,5 +283,5 @@
             <parent link="r_hip_pitch_link"/>
             <child link="r_knee_pitch_link"/>
-            <limit effort="10" lower="${-pi*0.9}" upper="${pi*0.9}" velocity="5.6548668"/>
+            <limit effort="20" lower="${-pi*0.9}" upper="${pi*0.9}" velocity="10"/>
             <dynamics damping="0.1" friction="0.0"/>
         </joint>
@@ -311,5 +311,5 @@
             <parent link="r_knee_pitch_link"/>
             <child link="r_ankle_pitch_link"/>
-            <limit effort="10" lower="${-pi*0.9}" upper="${pi*0.9}" velocity="5.6548668"/>
+            <limit effort="20" lower="${-pi*0.9}" upper="${pi*0.9}" velocity="10"/>
             <dynamics damping="0.1" friction="0.0"/>
         </joint>
@@ -339,5 +339,5 @@
             <parent link="r_ankle_pitch_link"/>
             <child link="r_ankle_roll_link"/>
-            <limit effort="10" lower="${-pi*0.9}" upper="${pi*0.9}" velocity="5.6548668"/>
+            <limit effort="20" lower="${-pi*0.9}" upper="${pi*0.9}" velocity="10"/>
             <dynamics damping="0.1" friction="0.0"/>
         </joint>
@@ -356,7 +356,7 @@
             </visual>
             <inertial>
-                <origin xyz="0.03576926 -0.08779574 -0.00045842"/>
+                            <origin xyz="0.03625957 -0.00019537 0.00037602"/>
                 <mass value="0.10500000"/>
-                <inertia ixx="0.00123572" ixy="0.00000500" ixz="0.00000812" iyy="0.00031773" iyz="0.00000828" izz="0.00094763" />
+                <inertia ixx="0.00034590" ixy="-0.00000013" ixz="0.00000857" iyy="0.00032704" iyz="0.00000120" izz="0.00004812" />
             </inertial>
         </link>
