Commit message: add urdf file

File: uthai_description/urdf/materials.xacro (robot description, xacro)
@@ -11,5 +11,5 @@
     </material>
     <material name="grey">
-        <color rgba="0.2 0.2 0.2 1.0"/>
+        <color rgba="0.4 0.4 0.4 1.0"/>
     </material>
     <material name="orange">

File: uthai_description/urdf/uthai.xacro (robot description, xacro)
@@ -5,8 +5,9 @@
     <!-- Import Rviz colors -->
     <xacro:include filename="$(find uthai_description)/urdf/materials.xacro" />
+    <xacro:include filename="$(find uthai_description)/urdf/uthai_leg.xacro" />
     <!-- Used for fixing robot -->
     <link name="world"></link>
     <joint name="world_fixed" type="fixed">
-        <origin xyz="0 0 0.75" rpy="0 0 0"/>
+        <origin xyz="0 0 0.756" rpy="0 0 0"/>
         <parent link="world"/>
         <child link="base"/>
@@ -34,8 +35,7 @@
         </visual>
         <inertial>
-            <origin xyz="0 0 0" rpy="0 0 0"/>
-            <mass value="6.869"/>
-            <inertia ixx="1.0" ixy="0.0" ixz="0.0" iyy="1.0" iyz="0.0" izz="1.0" />
-            <!--<inertia ixx="0.03603" ixy="0.0" ixz="0.00016" iyy="0.02210" iyz="0.0" izz="0.03830" />-->
+            <origin xyz="-0.00562901 0.00000232 -0.02326557"/>
+            <mass value="0.664564"/>
+            <inertia ixx="0.00504607" ixy="-0.00000002" ixz="-0.00000322" iyy="0.00052209" iyz="0.00000002" izz="0.00510184" />
         </inertial>
     </link>
@@ -47,3 +47,5 @@
     </joint>
     <link name="imu_link"></link>
+    <xacro:uthai_left_leg parent="pelvis_link"/>
+    <xacro:uthai_right_leg parent="pelvis_link"/>
 </robot>

Commit message: update xacro files

File: uthai_description/urdf/materials.xacro (robot description, xacro)
@@ -11,5 +11,5 @@
     </material>
     <material name="grey">
-        <color rgba="0.4 0.4 0.4 1.0"/>
+        <color rgba="0.6 0.6 0.6 1.0"/>
     </material>
     <material name="orange">

File: uthai_description/urdf/uthai.gazebo.xacro (robot description, xacro)
@@ -1,9 +1,10 @@
 <?xml version="1.0"?>
-<robot>
+<robot
+    xmlns:xacro="http://ros.org/wiki/xacro">
     <!-- ros_control plugin -->
     <gazebo>
         <plugin name="gazebo_ros_control" filename="libgazebo_ros_control.so">
             <robotNamespace>/uthai</robotNamespace>
-            <robotSimType>gazebo_ros_control/DefaultRobotHWSim</robotSimType>
+            <!-- <robotSimType>gazebo_ros_control/DefaultRobotHWSim</robotSimType> -->
         </plugin>
     </gazebo>
@@ -16,51 +17,25 @@
         </plugin>
     </gazebo>
-    <!-- <gazebo>
-        <plugin name="imu_plugin" filename="libgazebo_ros_imu.so">
-            <alwaysOn>true</alwaysOn>
-            <bodyName>imu_link</bodyName>
-            <topicName>/uthai/sensor/imu</topicName>
-            <serviceName>imu_service</serviceName>
-            <gaussianNoise>0.0</gaussianNoise>
-            <updateRate>10.0</updateRate>
-            <imu>
-                <noise>
-                    <type>gaussian</type>
-                    <rate>
-                        <mean>0.0</mean>
-                        <stddev>2e-4</stddev>
-                        <bias_mean>0.0000075</bias_mean>
-                        <bias_stddev>0.0000008</bias_stddev>
-                    </rate>
-                    <accel>
-                        <mean>0.0</mean>
-                        <stddev>1.7e-2</stddev>
-                        <bias_mean>0.1</bias_mean>
-                        <bias_stddev>0.001</bias_stddev>
-                    </accel>
-                </noise>
-            </imu>
-        </plugin>
-    </gazebo>-->
+    <!-- <gazebo><plugin name="imu_plugin" filename="libgazebo_ros_imu.so"><alwaysOn>true</alwaysOn><bodyName>imu_link</bodyName><topicName>/uthai/sensor/imu</topicName><serviceName>imu_service</serviceName><gaussianNoise>0.0</gaussianNoise><updateRate>10.0</updateRate><imu><noise><type>gaussian</type><rate><mean>0.0</mean><stddev>2e-4</stddev><bias_mean>0.0000075</bias_mean><bias_stddev>0.0000008</bias_stddev></rate><accel><mean>0.0</mean><stddev>1.7e-2</stddev><bias_mean>0.1</bias_mean><bias_stddev>0.001</bias_stddev></accel></noise></imu></plugin></gazebo>-->
     <!-- imu sensor -->
-  <gazebo reference="imu_link">
-    <gravity>true</gravity>
-    <sensor name="imu_sensor" type="imu">
-      <always_on>true</always_on>
-      <update_rate>100</update_rate>
-      <visualize>true</visualize>
-      <topic>/uthai/sensor/imu</topic>
-      <plugin filename="libgazebo_ros_imu_sensor.so" name="imu_plugin">
-        <topicName>uthai/sensor/imu</topicName>
-        <bodyName>imu_link</bodyName>
-        <updateRateHZ>10.0</updateRateHZ>
-        <gaussianNoise>0.0</gaussianNoise>
-        <xyzOffset>0 0 0</xyzOffset>
-        <rpyOffset>0 0 0</rpyOffset>
-        <frameName>imu_link</frameName>
-      </plugin>
-      <pose>0 0 0 0 0 0</pose>
-    </sensor>
-  </gazebo>
+    <gazebo reference="imu_link">
+        <gravity>true</gravity>
+        <sensor name="imu_sensor" type="imu">
+            <always_on>true</always_on>
+            <update_rate>100</update_rate>
+            <visualize>true</visualize>
+            <topic>/uthai/sensor/imu</topic>
+            <plugin filename="libgazebo_ros_imu_sensor.so" name="imu_plugin">
+                <topicName>uthai/sensor/imu</topicName>
+                <bodyName>imu_link</bodyName>
+                <updateRateHZ>10.0</updateRateHZ>
+                <gaussianNoise>0.0</gaussianNoise>
+                <xyzOffset>0 0 0</xyzOffset>
+                <rpyOffset>0 0 0</rpyOffset>
+                <frameName>imu_link</frameName>
+            </plugin>
+            <pose>0 0 0 0 0 0</pose>
+        </sensor>
+    </gazebo>
     <!-- World -->
     <gazebo reference="world"></gazebo>
@@ -71,33 +46,39 @@
     <!-- Body-->
     <gazebo reference="pelvis_link">
-         <mu1>0.2</mu1>
+        <mu1>0.2</mu1>
         <mu2>0.2</mu2>
         <material>Gazebo/Grey</material>
+        <selfCollide>false</selfCollide>
     </gazebo>
     <!-- Left Leg -->
     <gazebo reference="l_hip_yaw_link">
-           <mu1>0.2</mu1>
+        <mu1>0.2</mu1>
         <mu2>0.2</mu2>
         <material>Gazebo/Grey</material>
+        <selfCollide>false</selfCollide>
     </gazebo>
     <gazebo reference="l_hip_roll_link">
-           <mu1>0.2</mu1>
+        <mu1>0.2</mu1>
         <mu2>0.2</mu2>
         <material>Gazebo/Grey</material>
+        <selfCollide>false</selfCollide>
     </gazebo>
     <gazebo reference="l_hip_pitch_link">
-           <mu1>0.2</mu1>
+        <mu1>0.2</mu1>
         <mu2>0.2</mu2>
         <material>Gazebo/Grey</material>
+        <selfCollide>false</selfCollide>
     </gazebo>
     <gazebo reference="l_knee_pitch_link">
-           <mu1>0.2</mu1>
+        <mu1>0.2</mu1>
         <mu2>0.2</mu2>
         <material>Gazebo/Grey</material>
+        <selfCollide>false</selfCollide>
     </gazebo>
     <gazebo reference="l_ankle_pitch_link">
-          <mu1>0.2</mu1>
+        <mu1>0.2</mu1>
         <mu2>0.2</mu2>
         <material>Gazebo/Grey</material>
+        <selfCollide>false</selfCollide>
     </gazebo>
     <gazebo reference="l_ankle_roll_link">
@@ -108,32 +89,37 @@
         <fdir1>1 0 0</fdir1>
         <maxVel>1.0</maxVel>
-        <minDepth>0.0</minDepth>
+        <minDepth>0.001</minDepth>
         <material>Gazebo/Grey</material>
     </gazebo>
     <!-- Right Leg -->
     <gazebo reference="r_hip_yaw_link">
-       <mu1>0.2</mu1>
+        <mu1>0.2</mu1>
         <mu2>0.2</mu2>
         <material>Gazebo/Grey</material>
+        <selfCollide>false</selfCollide>
     </gazebo>
     <gazebo reference="r_hip_roll_link">
-           <mu1>0.2</mu1>
+        <mu1>0.2</mu1>
         <mu2>0.2</mu2>
         <material>Gazebo/Grey</material>
+        <selfCollide>false</selfCollide>
     </gazebo>
     <gazebo reference="r_hip_pitch_link">
-          <mu1>0.2</mu1>
+        <mu1>0.2</mu1>
         <mu2>0.2</mu2>
         <material>Gazebo/Grey</material>
+        <selfCollide>false</selfCollide>
     </gazebo>
     <gazebo reference="r_knee_pitch_link">
-         <mu1>0.2</mu1>
+        <mu1>0.2</mu1>
         <mu2>0.2</mu2>
         <material>Gazebo/Grey</material>
+        <selfCollide>false</selfCollide>
     </gazebo>
     <gazebo reference="r_ankle_pitch_link">
-           <mu1>0.2</mu1>
+        <mu1>0.2</mu1>
         <mu2>0.2</mu2>
         <material>Gazebo/Grey</material>
+        <selfCollide>false</selfCollide>
     </gazebo>
     <gazebo reference="r_ankle_roll_link">

File: uthai_description/urdf/uthai.xacro (robot description, xacro)
@@ -5,13 +5,13 @@
     <!-- Import Rviz colors -->
     <xacro:include filename="$(find uthai_description)/urdf/materials.xacro" />
-    <xacro:include filename="$(find uthai_description)/urdf/uthai_leg.xacro" />
-    <xacro:include filename="$(find uthai_description)/urdf/uthai.gazebo" />
+    <xacro:include filename="$(find uthai_description)/urdf/uthai.visuals.xacro" />
+    <xacro:include filename="$(find uthai_description)/urdf/uthai.inertia.xacro" />
+    <xacro:include filename="$(find uthai_description)/urdf/uthai.transmissions.xacro" />
+    <xacro:include filename="$(find uthai_description)/urdf/uthai.right_leg.xacro" />
+    <xacro:include filename="$(find uthai_description)/urdf/uthai.left_leg.xacro" />
+    <xacro:include filename="$(find uthai_description)/urdf/uthai.gazebo.xacro" />
     <!-- Used for fixing robot -->
-    <!--<link name="world"></link>
-    <joint name="world_fixed" type="fixed">
-        <origin xyz="0 0 0.756" rpy="0 0 0"/>
-        <parent link="world"/>
-        <child link="base"/>
-    </joint>
+    <link name="world"></link>
+    <!-- <joint name="world_fixed" type="fixed"><origin xyz="0 0 0.756" rpy="0 0 0"/><parent link="world"/><child link="base"/></joint> -->
     <link name="base"></link>
     <joint name="base_fixed" type="fixed">
@@ -19,24 +19,15 @@
         <parent link="base"/>
         <child link="pelvis_link"/>
-    </joint>-->
+    </joint>
     <!-- pelvis_link -->
     <link name="pelvis_link">
+        <visual>
+            <xacro:insert_mesh_pelvis_link />
+        </visual>
         <collision>
-            <origin xyz="0 0 0" rpy="0 0 0"/>
-            <geometry>
-                <mesh filename="package://uthai_description/meshes/pelvis.STL"/>
-            </geometry>
+            <xacro:insert_mesh_pelvis_link />
         </collision>
-        <visual>
-            <origin xyz="0 0 0" rpy="0 0 0"/>
-            <geometry>
-                <mesh filename="package://uthai_description/meshes/pelvis.STL"/>
-            </geometry>
-            <material name="grey"/>
-        </visual>
         <inertial>
-            <origin xyz="-0.00562901 0.00000232 -0.02326557"/>
-            <mass value="0.664564"/>
-            <inertia ixx="0.00504607" ixy="-0.00000002" ixz="-0.00000322" iyy="0.00052209" iyz="0.00000002" izz="0.00510184" />
+            <xacro:insert_inertia_pelvis_link />
         </inertial>
     </link>
@@ -48,5 +39,6 @@
     </joint>
     <link name="imu_link"></link>
+    <!-- leg link -->
+    <xacro:uthai_right_leg parent="pelvis_link"/>
     <xacro:uthai_left_leg parent="pelvis_link"/>
-    <xacro:uthai_right_leg parent="pelvis_link"/>
 </robot>
