Commit message: update parameter

File: uthai_description/urdf/model.urdf (robot description, URDF)
Before this commit: robot uthai, 17 links, 16 joints
Links:
- removed link base
- removed link pelvis_link
- added link base_footprint, mass 0.664564; collision mesh filename=package://uthai_description/meshes/base.STL scale=1 1 1; visual mesh filename=package://uthai_description/meshes/base.STL scale=1 1 1
- added link base_link
- link l_ankle_pitch_link: mass 0.34300000 -> 0.34200000
- link l_ankle_roll_link: mass 0.10500000 -> 0.155
- link l_hip_pitch_link: mass 0.31800000 -> 0.33732478
- link l_hip_roll_link: mass 0.34300000 -> 0.342
- link l_hip_yaw_link: mass 0.09100000 -> 0.090718
- link r_ankle_pitch_link: mass 0.34300000 -> 0.342
- link r_ankle_roll_link: mass 0.10500000 -> 0.155
- link r_hip_pitch_link: mass 0.31800000 -> 0.33732478
- link r_hip_roll_link: mass 0.34300000 -> 0.342
- link r_hip_yaw_link: mass 0.09100000 -> 0.090718
Joints:
- joint base_fixed: child pelvis_link -> base_footprint; parent base -> base_link
- joint imu_fixed: parent pelvis_link -> base_footprint
- joint l_ankle_pitch_joint: limit lower=-2.8274333886 upper=2.8274333886 effort=1000 velocity=5 -> lower=-2.8274333886 upper=2.8274333886 effort=1000 velocity=3
- joint l_ankle_roll_joint: limit lower=-2.8274333886 upper=2.8274333886 effort=1000 velocity=5 -> lower=-2.8274333886 upper=2.8274333886 effort=1000 velocity=3
- joint l_ft_fixed: origin xyz=0.05 0.0 0.0 rpy=0 -1.570796327 0 -> xyz=0.045 0.0 0.0 rpy=0 -1.570796327 0
- joint l_hip_pitch_joint: limit lower=-2.8274333886 upper=2.8274333886 effort=1000 velocity=5 -> lower=-2.8274333886 upper=2.8274333886 effort=1000 velocity=3; origin xyz=0 0 -0.005 rpy=-1.570796327 0 -1.570796327 -> xyz=0 0 0 rpy=-1.570796327 0 -1.570796327
- joint l_hip_roll_joint: limit lower=-2.8274333886 upper=2.8274333886 effort=1000 velocity=5 -> lower=-2.8274333886 upper=2.8274333886 effort=1000 velocity=3
- joint l_hip_yaw_joint: limit lower=-2.8274333886 upper=2.8274333886 effort=1000 velocity=5 -> lower=-2.8274333886 upper=2.8274333886 effort=1000 velocity=3; origin xyz=0.008 0.09 -0.06 rpy=0 0 1.570796327 -> xyz=0.0 0.09 -0.068 rpy=0 0 1.570796327; parent pelvis_link -> base_footprint
- joint l_knee_pitch_joint: limit lower=-2.8274333886 upper=2.8274333886 effort=1000 velocity=5 -> lower=-2.8274333886 upper=2.8274333886 effort=1000 velocity=3
- joint r_ankle_pitch_joint: limit lower=-2.8274333886 upper=2.8274333886 effort=1000 velocity=5 -> lower=-2.8274333886 upper=2.8274333886 effort=1000 velocity=3
- joint r_ankle_roll_joint: limit lower=-2.8274333886 upper=2.8274333886 effort=1000 velocity=5 -> lower=-2.8274333886 upper=2.8274333886 effort=1000 velocity=3
- joint r_ft_fixed: origin xyz=0.05 0.0 0.0 rpy=0 -1.570796327 0 -> xyz=0.045 0.0 0.0 rpy=0 -1.570796327 0
- joint r_hip_pitch_joint: limit lower=-2.8274333886 upper=2.8274333886 effort=1000 velocity=5 -> lower=-2.8274333886 upper=2.8274333886 effort=1000 velocity=3; origin xyz=0 0 -0.005 rpy=-1.570796327 0 -1.570796327 -> xyz=0 0 0 rpy=-1.570796327 0 -1.570796327
- joint r_hip_roll_joint: limit lower=-2.8274333886 upper=2.8274333886 effort=1000 velocity=5 -> lower=-2.8274333886 upper=2.8274333886 effort=1000 velocity=3
- joint r_hip_yaw_joint: limit lower=-2.8274333886 upper=2.8274333886 effort=1000 velocity=5 -> lower=-2.8274333886 upper=2.8274333886 effort=1000 velocity=3; origin xyz=0.008 -0.09 -0.06 rpy=0 0 -1.570796327 -> xyz=0.0 -0.09 -0.068 rpy=0 0 -1.570796327; parent pelvis_link -> base_footprint
- joint r_knee_pitch_joint: limit lower=-2.8274333886 upper=2.8274333886 effort=1000 velocity=5 -> lower=-2.8274333886 upper=2.8274333886 effort=1000 velocity=3

File: uthai_description/urdf/uthai.gazebo.xacro (robot description, xacro)
@@ -6,12 +6,11 @@
         <plugin name="gazebo_ros_control" filename="libgazebo_ros_control.so">
             <robotNamespace>/uthai</robotNamespace>
-            <!-- <robotSimType>gazebo_ros_control/DefaultRobotHWSim</robotSimType> -->
-        </plugin>
+         </plugin>
     </gazebo>
     <gazebo>
         <plugin name="ground_truth" filename="libgazebo_ros_p3d.so">
             <frameName>map</frameName>
-            <bodyName>pelvis_link</bodyName>
-            <topicName>odom</topicName>
+            <bodyName>base_link</bodyName>
+            <topicName>/uthai/odom</topicName>
             <updateRate>100.0</updateRate>
         </plugin>
@@ -40,10 +39,12 @@
     <!-- World -->
     <gazebo reference="world"></gazebo>
+    <!-- Map -->
+    <gazebo reference="map"></gazebo>
     <!-- Base -->
-    <gazebo reference="base"></gazebo>
+    <gazebo reference="base_link"></gazebo>
     <!-- IMU -->
     <gazebo reference="imu_link"></gazebo>
     <!-- Body-->
-    <gazebo reference="pelvis_link">
+    <gazebo reference="base_footprint">
         <mu1>0.2</mu1>
         <mu2>0.2</mu2>
@@ -83,13 +84,13 @@
     </gazebo>
     <gazebo reference="l_ankle_roll_link">
-        <kp>100000.0</kp>
+         <kp>100000.0</kp>
         <kd>100.0</kd>
-        <mu1>0.6</mu1>
-        <mu2>0.6</mu2>
-        <maxContacts>3</maxContacts>
-        <fdir1>1 1 1</fdir1>
-        <!-- <maxVel>1.0</maxVel> -->
+        <mu1>1.5</mu1>
+        <mu2>1.5</mu2>
+        <!--<maxContacts>30</maxContacts>-->
+        <fdir1>1 1 0</fdir1>
+        <maxVel>1.0</maxVel>
         <minDepth>0.001</minDepth>
-        <material>Gazebo/Grey</material>
+        <material>Gazebo/Blue</material>
     </gazebo>
     <!-- Right Leg -->
@@ -127,12 +128,11 @@
         <kp>100000.0</kp>
         <kd>100.0</kd>
-        <mu1>0.6</mu1>
-        <!-- <mu2>1.5</mu2> -->
-        <mu2>0.6</mu2>
-        <maxContacts>3</maxContacts>
-        <fdir1>1 1 1</fdir1>
-        <!-- <maxVel>1.0</maxVel> -->
+        <mu1>1.5</mu1>
+        <mu2>1.5</mu2>
+        <!--<maxContacts>30</maxContacts>-->
+        <fdir1>1 1 0</fdir1>
+         <maxVel>1.0</maxVel>
         <minDepth>0.0001</minDepth>
-        <material>Gazebo/Grey</material>
+        <material>Gazebo/Blue</material>
     </gazebo>
 </robot>

File: uthai_description/urdf/uthai.inertia.xacro (robot description, xacro)
@@ -3,80 +3,80 @@
     xmlns:xacro="http://www.ros.org/wiki/xacro">
     <!-- body link -->
-    <xacro:macro name="insert_inertia_pelvis_link">
-        <origin xyz="-0.00557436 0.00000000 -0.02356598"/>
-        <mass value="0.86500000"/>
-        <inertia ixx="0.00656431" ixy="-0.00000003" ixz="-0.00000466" iyy="0.00067608" iyz="0.00000000" izz="0.00664141" />
+    <xacro:macro name="insert_inertia_base_link">
+        <origin xyz="-0.00856879 0.00000000 -0.02356598"/>
+        <mass value="0.664564"/>
+        <inertia ixx="0.00504324" ixy="-0.00000002" ixz="-0.00000358" iyy="0.00051942" iyz="0.00000000" izz="0.00510248" />
     </xacro:macro>
     <!-- right hip yaw link -->
     <xacro:macro name="insert_inertia_r_hip_yaw_link">
-        <origin xyz="0.00000000 -0.02500000 -0.00735017" />
-        <mass value="0.09100000"/>
-        <inertia ixx="0.00014158" ixy="0.00000000" ixz="0.00000000" iyy="0.00002022" iyz="0.00000000" izz="0.00014316" />
+        <origin xyz="0.00000000 -0.01999 -0.00735017" />
+        <mass value="0.090718"/>
+        <inertia ixx="0.00014114" ixy="0.00000000" ixz="0.00000000" iyy="0.00002016" iyz="0.00000000" izz="0.00014272" />
     </xacro:macro>
     <!-- right hip roll link -->
     <xacro:macro name="insert_inertia_r_hip_roll_link">
-        <origin xyz="0.00000000 -0.01526210 -0.02652545" />
-        <mass value="0.34300000"/>
-        <inertia ixx="0.00032449" ixy="0.00000081" ixz="0.00000000" iyy="0.00026847" iyz="0.00000219" izz="0.00014760" />
+        <origin xyz="-0.00005878 -0.01433229 -0.01958936" />
+        <mass value="0.342"/>
+        <inertia ixx="0.00033963" ixy="0.00000054" ixz="-0.00000042" iyy="0.00029059" iyz="0.00001145" izz="0.00015024" />
     </xacro:macro>
     <!-- right hip pitch link -->
     <xacro:macro name="insert_inertia_r_hip_pitch_link">
-        <origin xyz="0.22137989 0.00000000 0.00000000" />
-        <mass value="0.31800000"/>
-        <inertia ixx="0.00011525" ixy="0.00000000" ixz="0.00000078" iyy="0.00254669" iyz="0.00000000" izz="0.00250848" />
+        <origin xyz="0.21422113 0.0 0.0" />
+        <mass value="0.33732478"/>
+        <inertia ixx="0.00012533" ixy="0.00000000" ixz="0.00000079" iyy="0.00295762" iyz="0.00000000" izz="0.00291401" />
     </xacro:macro>
     <!-- right knee link -->
     <xacro:macro name="insert_inertia_r_knee_pitch_link">
-        <origin xyz="0.16288218 0.00000000 0.00000000" />
+        <origin xyz="0.16288151 0.00000000 0.00000000" />
         <mass value="0.15100000"/>
-        <inertia ixx="0.00006340" ixy="0.0" ixz="0.0" iyy="0.00139612" iyz="0.0" izz="0.00136731" />
+        <inertia ixx="0.0000634" ixy="0.0" ixz="0.0" iyy="0.00139615" iyz="0.0" izz="0.00136734" />
     </xacro:macro>
     <!-- right ankle pitch link -->
     <xacro:macro name="insert_inertia_r_ankle_pitch_link">
-        <origin xyz="-0.01526210 0.02152545 0.00000000" />
-        <mass value="0.34300000"/>
-        <inertia ixx="0.00026847" ixy="-0.00000219" ixz="-0.00000081" iyy="0.00014760" iyz="0.00000000" izz="0.00032449" />
+        <origin xyz="-0.01433229 0.01958936 0.00005878" />
+        <mass value="0.342"/>
+        <inertia ixx="0.00029059" ixy="-0.00001145" ixz="-0.00000054" iyy="0.00015024" iyz="-0.00000042" izz="0.00033963" />
     </xacro:macro>
     <!-- right ankle roll link -->
     <xacro:macro name="insert_inertia_r_ankle_roll_link">
-        <origin xyz="0.03625882 -0.00019548 0.00034576" />
-        <mass value="0.10500000"/>
-        <inertia ixx="0.00034591" ixy="-0.00000013" ixz="0.00000857" iyy="0.00032705" iyz="0.00000120" izz="0.00004813" />
+        <origin xyz="0.03627101 -0.00000116 0.00053793" />
+        <mass value="0.155"/>
+        <inertia ixx="0.00052206" ixy="0" ixz="0.00001" iyy="0.00047025" iyz="0" izz="0.00009087" />
     </xacro:macro>
     <!-- left hip yaw link -->
     <xacro:macro name="insert_inertia_l_hip_yaw_link">
-        <origin xyz="0.00000000 0.02500000 -0.00735017" />
-        <mass value="0.09100000"/>
-        <inertia ixx="0.00014158" ixy="0.0" ixz="0.0" iyy="0.00002022" iyz="0.0" izz="0.00014316" />
+        <origin xyz="0 0.01999 -0.00735017" />
+        <mass value="0.090718"/>
+        <inertia ixx="0.00014114" ixy="0.0" ixz="0.0" iyy="0.00002016" iyz="0.0" izz="0.00014272" />
     </xacro:macro>
     <!-- left hip roll link -->
     <xacro:macro name="insert_inertia_l_hip_roll_link">
-        <origin xyz="0.00000000 -0.01526210 -0.02652545" />
-        <mass value="0.34300000"/>
-        <inertia ixx="0.00032449" ixy="-0.00000081" ixz="0.00000000" iyy="0.00026847" iyz="0.00000219" izz="0.00014760" />
+        <origin xyz="-0.00005878 -0.01433229 -0.01958936" />
+        <mass value="0.342"/>
+        <inertia ixx="0.00033963" ixy="0.00000054" ixz="-0.00000042" iyy="0.00029059" iyz="0.00001145" izz="0.00015024" />
     </xacro:macro>
     <!-- left hip pitch link -->
     <xacro:macro name="insert_inertia_l_hip_pitch_link">
-        <origin xyz="0.22137989 0.00000000 0.00000000" />
-        <mass value="0.31800000"/>
-        <inertia ixx="0.00011525" ixy="0.00000000" ixz="0.00000078" iyy="0.00254669" iyz="0.00000000" izz="0.00250848" />
+        <origin xyz="0.21422113 0.00000000 0.00000000" />
+        <mass value="0.33732478"/>
+        <inertia ixx="0.00012533" ixy="0.00000000" ixz="0.00000079" iyy="0.00295762" iyz="0.00000000" izz="0.00291401" />
     </xacro:macro>
     <!-- left knee link -->
     <xacro:macro name="insert_inertia_l_knee_pitch_link">
-        <origin xyz="0.16288218 0.00000000 0.00000000" />
+        <origin xyz="0.16288151 0.00000000 0.00000000" />
         <mass value="0.15100000"/>
-        <inertia ixx="0.00006340" ixy="0.0" ixz="0.0" iyy="0.00139612" iyz="0.0" izz="0.00136731" />
+        <inertia ixx="0.0000634" ixy="0.0" ixz="0.0" iyy="0.00139615" iyz="0.0" izz="0.00136734" />
     </xacro:macro>
     <!-- left ankle pitch link -->
     <xacro:macro name="insert_inertia_l_ankle_pitch_link">
-        <origin xyz="-0.01526210 0.02152545 0.00000000" />
-        <mass value="0.34300000"/>
-        <inertia ixx="0.00026847" ixy="-0.00000219" ixz="-0.00000081" iyy="0.00014760" iyz="0.00000000" izz="0.00032449" />
+        <origin xyz="-0.01433229 0.01958936 0.00005878" />
+        <mass value="0.34200000"/>
+        <inertia ixx="0.00029059" ixy="-0.00001145" ixz="-0.00000054" iyy="0.00015024" iyz="-0.00000042" izz="0.00033963" />
     </xacro:macro>
     <!-- left ankle roll link -->
     <xacro:macro name="insert_inertia_l_ankle_roll_link">
-        <origin xyz="0.03608455 0.00020160 0.00002697" />
-        <mass value="0.10500000"/>
-        <inertia ixx="0.00034223" ixy="0.00000014" ixz="0.00000840" iyy="0.00032348" iyz="-0.00000118" izz="0.00004816" />
+        <origin xyz="0.03627101 -0.00000116 0.00053793" />
+        <mass value="0.155"/>
+        <inertia ixx="0.00052206" ixy="0.000000" ixz="0.00001" iyy="0.00047025" iyz="0" izz="0.00009087" />
     </xacro:macro>
 </robot>

File: uthai_description/urdf/uthai.left_leg.xacro (robot description, xacro)
@@ -3,12 +3,12 @@
     xmlns:xacro="http://www.ros.org/wiki/xacro">
     <!-- left leg -->
-    <xacro:macro name="uthai_left_leg" params="parent">
+    <xacro:macro name="uthai_left_leg" params="parent dxl_effort dxl_speed">
         <!-- left hip yaw joint -->
         <joint name="l_hip_yaw_joint" type="revolute">
             <axis xyz="0 0 1" />
-            <origin xyz="0.008 0.09 -0.06" rpy="0 0 ${pi/2}"/>
+            <origin xyz="0.0 0.09 -0.068" rpy="0 0 ${pi/2}"/>
             <parent link="${parent}"/>
             <child link="l_hip_yaw_link"/>
-            <limit effort="1000" lower="${-pi*0.9}" upper="${pi*0.9}" velocity="5"/>
+            <limit effort="${dxl_effort}" lower="${-pi*0.9}" upper="${pi*0.9}" velocity="${dxl_speed}"/>
             <dynamics damping="0.1" friction="0.0"/>
         </joint>
@@ -32,5 +32,5 @@
             <parent link="l_hip_yaw_link"/>
             <child link="l_hip_roll_link"/>
-            <limit effort="1000" lower="${-pi*0.9}" upper="${pi*0.9}" velocity="5"/>
+            <limit effort="${dxl_effort}" lower="${-pi*0.9}" upper="${pi*0.9}" velocity="${dxl_speed}"/>
             <dynamics damping="0.1" friction="0.0"/>
         </joint>
@@ -51,8 +51,8 @@
         <joint name="l_hip_pitch_joint" type="revolute">
             <axis xyz="0 0 1" />
-            <origin xyz="0 0 -0.005" rpy="${-pi/2} 0 ${-pi/2}"/>
+            <origin xyz="0 0 0" rpy="${-pi/2} 0 ${-pi/2}"/>
             <parent link="l_hip_roll_link"/>
             <child link="l_hip_pitch_link"/>
-            <limit effort="1000" lower="${-pi*0.9}" upper="${pi*0.9}" velocity="5"/>
+            <limit effort="${dxl_effort}" lower="${-pi*0.9}" upper="${pi*0.9}" velocity="${dxl_speed}"/>
             <dynamics damping="0.1" friction="0.0"/>
         </joint>
@@ -76,5 +76,5 @@
             <parent link="l_hip_pitch_link"/>
             <child link="l_knee_pitch_link"/>
-            <limit effort="1000" lower="${-pi*0.9}" upper="${pi*0.9}" velocity="5"/>
+            <limit effort="${dxl_effort}" lower="${-pi*0.9}" upper="${pi*0.9}" velocity="${dxl_speed}"/>
             <dynamics damping="0.1" friction="0.0"/>
         </joint>
@@ -98,5 +98,5 @@
             <parent link="l_knee_pitch_link"/>
             <child link="l_ankle_pitch_link"/>
-            <limit effort="1000" lower="${-pi*0.9}" upper="${pi*0.9}" velocity="5"/>
+            <limit effort="${dxl_effort}" lower="${-pi*0.9}" upper="${pi*0.9}" velocity="${dxl_speed}"/>
             <dynamics damping="0.1" friction="0.0"/>
         </joint>
@@ -120,5 +120,5 @@
             <parent link="l_ankle_pitch_link"/>
             <child link="l_ankle_roll_link"/>
-            <limit effort="1000" lower="${-pi*0.9}" upper="${pi*0.9}" velocity="5"/>
+            <limit effort="${dxl_effort}" lower="${-pi*0.9}" upper="${pi*0.9}" velocity="${dxl_speed}"/>
             <dynamics damping="0.1" friction="0.0"/>
         </joint>
@@ -138,5 +138,5 @@
         <!-- left ft fixed joint -->
         <joint name="l_ft_fixed" type="fixed">
-            <origin xyz="0.05 0.0 0.0" rpy="0 ${-pi/2} 0"/>
+            <origin xyz="0.045 0.0 0.0" rpy="0 ${-pi/2} 0"/>
             <parent link="l_ankle_roll_link"/>
             <child link="l_foot_ft_link"/>

File: uthai_description/urdf/uthai.right_leg.xacro (robot description, xacro)
@@ -3,12 +3,12 @@
     xmlns:xacro="http://www.ros.org/wiki/xacro">
     <!-- right leg -->
-    <xacro:macro name="uthai_right_leg" params="parent">
+    <xacro:macro name="uthai_right_leg" params="parent dxl_effort dxl_speed">
         <!-- right hip yaw joint -->
         <joint name="r_hip_yaw_joint" type="revolute">
             <axis xyz="0 0 1" />
-            <origin xyz="0.008 -0.09 -0.06" rpy="0 0 ${-pi/2}"/>
+            <origin xyz="0.0 -0.09 -0.068" rpy="0 0 ${-pi/2}"/>
             <parent link="${parent}"/>
             <child link="r_hip_yaw_link"/>
-            <limit effort="1000" lower="${-pi*0.9}" upper="${pi*0.9}" velocity="5"/>
+            <limit effort="${dxl_effort}" lower="${-pi*0.9}" upper="${pi*0.9}" velocity="${dxl_speed}"/>
             <dynamics damping="0.1" friction="0.0"/>
         </joint>
@@ -32,5 +32,5 @@
             <parent link="r_hip_yaw_link"/>
             <child link="r_hip_roll_link"/>
-            <limit effort="1000" lower="${-pi*0.9}" upper="${pi*0.9}" velocity="5"/>
+            <limit effort="${dxl_effort}" lower="${-pi*0.9}" upper="${pi*0.9}" velocity="${dxl_speed}"/>
             <dynamics damping="0.1" friction="0.0"/>
         </joint>
@@ -51,8 +51,8 @@
         <joint name="r_hip_pitch_joint" type="revolute">
             <axis xyz="0 0 1" />
-            <origin xyz="0 0 -0.005" rpy="${-pi/2} 0 ${-pi/2}"/>
+            <origin xyz="0 0 0" rpy="${-pi/2} 0 ${-pi/2}"/>
             <parent link="r_hip_roll_link"/>
             <child link="r_hip_pitch_link"/>
-            <limit effort="1000" lower="${-pi*0.9}" upper="${pi*0.9}" velocity="5"/>
+            <limit effort="${dxl_effort}" lower="${-pi*0.9}" upper="${pi*0.9}" velocity="${dxl_speed}"/>
             <dynamics damping="0.1" friction="0.0"/>
         </joint>
@@ -76,5 +76,5 @@
             <parent link="r_hip_pitch_link"/>
             <child link="r_knee_pitch_link"/>
-            <limit effort="1000" lower="${-pi*0.9}" upper="${pi*0.9}" velocity="5"/>
+            <limit effort="${dxl_effort}" lower="${-pi*0.9}" upper="${pi*0.9}" velocity="${dxl_speed}"/>
             <dynamics damping="0.1" friction="0.0"/>
         </joint>
@@ -98,5 +98,5 @@
             <parent link="r_knee_pitch_link"/>
             <child link="r_ankle_pitch_link"/>
-            <limit effort="1000" lower="${-pi*0.9}" upper="${pi*0.9}" velocity="5"/>
+            <limit effort="${dxl_effort}" lower="${-pi*0.9}" upper="${pi*0.9}" velocity="${dxl_speed}"/>
             <dynamics damping="0.1" friction="0.0"/>
         </joint>
@@ -120,5 +120,5 @@
             <parent link="r_ankle_pitch_link"/>
             <child link="r_ankle_roll_link"/>
-            <limit effort="1000" lower="${-pi*0.9}" upper="${pi*0.9}" velocity="5"/>
+            <limit effort="${dxl_effort}" lower="${-pi*0.9}" upper="${pi*0.9}" velocity="${dxl_speed}"/>
             <dynamics damping="0.1" friction="0.0"/>
         </joint>
@@ -138,5 +138,5 @@
         <!-- right ft fixed joint -->
         <joint name="r_ft_fixed" type="fixed">
-            <origin xyz="0.05 0.0 0.0" rpy="0 ${-pi/2} 0"/>
+            <origin xyz="0.045 0.0 0.0" rpy="0 ${-pi/2} 0"/>
             <parent link="r_ankle_roll_link"/>
             <child link="r_foot_ft_link"/>

File: uthai_description/urdf/uthai.urdf.xacro (robot description, xacro)
@@ -3,5 +3,5 @@
     xmlns:xacro="http://www.ros.org/wiki/xacro">
     <xacro:property name="pi" value="3.141592654"/>
-    <!-- Import Rviz colors -->
+    <!-- Import xacro file -->
     <xacro:include filename="$(find uthai_description)/urdf/materials.xacro" />
     <xacro:include filename="$(find uthai_description)/urdf/uthai.visuals.xacro" />
@@ -12,33 +12,37 @@
     <xacro:include filename="$(find uthai_description)/urdf/uthai.gazebo.xacro" />
     <!-- Used for fixing robot -->
-    <!-- <link name="world"></link> -->
-    <!-- <joint name="world_fixed" type="fixed"><origin xyz="0 0 0.756" rpy="0 0 0"/><parent link="world"/><child link="base"/></joint> -->
-    <link name="base"></link>
+    <!--<link name="world"></link>
+    <joint name="world_fixed" type="fixed">
+        <origin xyz="0 0 0.764" rpy="0 0 0"/>
+        <parent link="world"/>
+        <child link="base_link"/>
+    </joint> -->
+    <link name="base_link"></link>
     <joint name="base_fixed" type="fixed">
         <origin xyz="0 0 0" rpy="0 0 0"/>
-        <parent link="base"/>
-        <child link="pelvis_link"/>
+        <parent link="base_link"/>
+        <child link="base_footprint"/>
     </joint>
-    <!-- pelvis_link -->
-    <link name="pelvis_link">
+    <!-- base_link -->
+    <link name="base_footprint">
         <visual>
-            <xacro:insert_mesh_pelvis_link />
+            <xacro:insert_mesh_base_link />
         </visual>
         <collision>
-            <xacro:insert_mesh_pelvis_link />
+            <xacro:insert_mesh_base_link />
         </collision>
         <inertial>
-            <xacro:insert_inertia_pelvis_link />
+            <xacro:insert_inertia_base_link />
         </inertial>
     </link>
     <!-- imu joint -->
     <joint name="imu_fixed" type="fixed">
-        <parent link="pelvis_link"/>
+        <origin xyz="0.0 0 0.45" rpy="0 0 0"/>
+        <parent link="base_footprint"/>
         <child link="imu_link"/>
-        <origin xyz="0.0 0 0.45" rpy="0 0 0"/>
     </joint>
     <link name="imu_link"></link>
     <!-- leg link -->
-    <xacro:uthai_right_leg parent="pelvis_link"/>
-    <xacro:uthai_left_leg parent="pelvis_link"/>
+    <xacro:uthai_right_leg parent="base_footprint" dxl_effort="1000" dxl_speed="3"/>
+    <xacro:uthai_left_leg parent="base_footprint" dxl_effort="1000" dxl_speed="3"/>
 </robot>

File: uthai_description/urdf/uthai.visuals.xacro (robot description, xacro)
@@ -3,8 +3,8 @@
     xmlns:xacro="http://www.ros.org/wiki/xacro">
     <!-- body link -->
-    <xacro:macro name="insert_mesh_pelvis_link">
+    <xacro:macro name="insert_mesh_base_link">
         <origin xyz="0 0 0" rpy="0 0 0" />
         <geometry>
-            <mesh filename="package://uthai_description/meshes/pelvis.STL" scale="1 1 1" />
+            <mesh filename="package://uthai_description/meshes/base.STL" scale="1 1 1" />
         </geometry>
         <material name="grey"/>
